File: KiCad/PWRBlock.sch (KiCad schematic (older format))
At the start: 26 parts

Commit message: Netztliste erstellt
Parts:
- removed D?: RED, symbol LED
- removed D? (x2): PURP, symbol LED
- removed D? (x2): BLUE, symbol LED
- removed P?: CONN_01X03, symbol CONN_01X03
- removed R? (x5): 330, symbol R
- added C1, C4, C6, C7: 100n, Capacitors_SMD:C_0805, symbol C
- added C2: 100µ, Capacitors_SMD:C_0805, symbol CP
- added C3: 47µ, Capacitors_ThroughHole:C_Radial_D10_L20_P2.5-5, symbol CP
- added C8: C, Capacitors_SMD:C_0805, symbol C
- added D1, D2: D, Diodes_SMD:SMA-SMB_Universal_Handsoldering, symbol D
- added D4, D5, D6, D7, D8: SMD-LED BC02, Sven:SMD_LED_4Pin_special, symbol LED_RGB
- added P1: CONN_02X02, Socket_Strips:Socket_Strip_Straight_2x02, symbol CONN_02X02
- added P4: CONN_02X04, Pin_Headers:Pin_Header_Straight_2x04, symbol CONN_02X04
- added Q1, Q2, Q3, Q4: Q_NMOS_GSD, TO_SOT_Packages_SMD:SOT-23_Handsoldering, symbol Q_NMOS_GSD
- added R10, R25, R26, R9: 10, Resistors_SMD:R_0805, symbol R
- added R11, R12, R13, R14: 10k, Resistors_SMD:R_0805, symbol R
- added R15, R16, R17, R18, R19, R20, R21, R22, R23, R24, R4, R6, R8: R, Resistors_SMD:R_0805, symbol R
- added R2: 1, Resistors_SMD:R_0805, symbol R
- added U1: AP1117, Toni:SOT223_GND_VO_VI, symbol AP1117
- C5: renamed from C?; value CP -> 47µ; footprint (none) -> Capacitors_ThroughHole:C_Radial_D10_L20_P2.5-5
- C9: renamed from C?; footprint (none) -> Capacitors_ThroughHole:C_Disc_D6_P5
- D3: renamed from D?; footprint (none) -> LEDs:LED-5MM
- F1: renamed from F?; footprint (none) -> Sven:Fuseholder5x20
- G1: renamed from G?; footprint (none) -> Socket_Strips:Socket_Strip_Straight_1x02
- IC1: renamed from IC?; footprint (none) -> PhilippsFootprints:Mini360
- IC2: renamed from IC?; footprint TQFP32 -> Housings_QFP:TQFP-32_7x7mm_Pitch0.8mm
- P2, P5: renamed from P?; footprint (none) -> Sven:Screw_Connector_5,08mm_x2
- R1: renamed from R?; value 330 -> 1k; footprint (none) -> Resistors_SMD:R_0805
- R27: renamed from R?; footprint (none) -> Resistors_ThroughHole:Resistor_Horizontal_RM15mm
- R3, R5, R7: renamed from R?; footprint (none) -> Resistors_SMD:R_0805
- S1: renamed from S?; footprint (none) -> Relays_ThroughHole:Relay_DPDT_Schrack-RT2_RM5mm
Connections:
- net +5V: now also R16.1, R18.1, R20.1, R21.1, R23.1, R4.1
- net GND: now also C1.2, C2.2, C3.2, C4.2, C6.2, C7.2, D4.1 (RC), D5.1 (RC), D6.1 (RC), D7.3 (BC), D8.3 (BC), P1.4 (P4), P4.2 (P2), P4.4 (P4), P4.6 (P6), P4.8 (P8), Q1.2 (S), Q2.2 (S), Q3.2 (S), Q4.2 (S), U1.1 (GND/ADJ); no longer S1.1 (N)
- net GNDA: now also C8.2, R6.2
- net VCC: now also R1.1, D1.2 (A), D2.2 (A), P1.2 (P2); no longer IC1.1 (Vin+)
- net at IC2.1 ((INT1)PD3): now also R22.1
- net at IC2.10 ((AIN0)PD6): now also R26.2
- net at IC2.12 ((ICP)PB0): now also R9.2
- net at IC2.13 ((OC1A)PB1): now also R10.2
- net Tab: now reaches IC2.14 ((~SS~/OC1B)PB2)
- net Tab: now also C7.1, P1.3 (P3), R8.2
- net MOSI: now reaches IC2.15 ((MOSI/OC2)PB3)
- net MISO: now reaches IC2.16 ((MISO)PB4)
- net SCK: now reaches IC2.17 ((SCK)PB5)
- net +5VA: now reaches IC2.18 (AVCC)
- net +5VA: now also IC2.4 (VCC), IC2.6 (VCC), S1.1 (N), C1.1, C2.1, C6.1, R8.1, U1.2 (VO)
- net Sens5V: now reaches IC2.19 (ADC6)
- net Sens5V: now also R4.2, R6.1
- net at IC2.2 ((XCK/T0)PD4): now also R24.1
- net at IC2.20 (AREF): now also C8.1
- net at IC2.23 ((ADC0)PC0): now also P4.1 (P1), R11.1
- net at IC2.24 ((ADC1)PC1): now also P4.3 (P3), R12.1
- net at IC2.25 ((ADC2)PC2): now also P4.5 (P5), R13.1
- net at IC2.26 ((ADC3)PC3): now also P4.7 (P7), R14.1
- net at IC2.27 ((ADC4/SDA)PC4): now also R11.2, R12.2, R13.2, R14.2
- net RES: now reaches IC2.29 (PC6(~RESET~))
- net at IC2.30 ((RXD)PD0): now also R15.1
- net at IC2.31 ((TXD)PD1): now also R17.1
- net at IC2.32 ((INT0)PD2): now also R19.1
- net at IC2.9 ((T1)PD5): now also R25.2; no longer R1.1
- net at F1.2, S1.1IN, S1.2IN: now also P1.1 (P1)
- net RelOff: now reaches S1.2 (L)
- net RelOff: now also Q2.3 (D)
- net RelOn: now reaches S1.3 (R)
- net RelOn: now also Q1.3 (D)
- new net: D1.1 (K), IC1.1 (Vin+)
- new net: D4.3 (BC), D5.3 (BC), D6.3 (BC), Q3.3 (D)
- new net: D4.4 (BA), R16.2
- new net: D4.6 (RA), R15.2
- new net: D5.4 (BA), R18.2
- new net: D5.6 (RA), R17.2
- new net: D6.4 (BA), R20.2
- new net: D6.6 (RA), R19.2
- new net: D7.1 (RC), D8.1 (RC), Q4.3 (D)
- new net: D7.4 (BA), R22.2
- new net: D7.6 (RA), R21.2
- new net: D8.4 (BA), R24.2
- new net: D8.6 (RA), R23.2
- new net: C3.1, C4.1, R2.1, U1.3 (VI)
- new net: D2.1 (K), R2.2
- new net: Q1.1 (G), R9.1
- new net: Q2.1 (G), R10.1
- new net AllBlue: Q3.1 (G), R26.1
- new net AllRed: Q4.1 (G), R25.1
- no-connect marks 2 -> 16
Other:
- moved on the sheet: C5, D3, F1, P2, R1, R7, S1

Commit message: Platienengröße geändert
Parts:
- added P3: CONN_02X04, Pin_Headers:Pin_Header_Straight_2x04, symbol CONN_02X04
- added P6: Pout1, Sven:Screw_Connector_5,08mm_x2, symbol CONN_01X02
- added P7: Pout2, Sven:Screw_Connector_5,08mm_x2, symbol CONN_01X02
- added R28, R29, R30, R31: 1k, Resistors_SMD:R_0805, symbol R
- added R32: 10, Resistors_SMD:R_0805, symbol R
- D4, D5, D6, D7, D8: footprint Sven:SMD_LED_4Pin_special -> LEDs2:LRTB_G6TG
Connections:
- net +5V: now also P7.2 (P2)
- net +5VA: now also P3.2 (P2), R32.1; no longer S1.1 (N)
- net AllBlue: now also R30.1
- net AllRed: now also R31.1
- net GND: now also P3.6 (P6), P6.2 (P2), R28.1, R29.2, R30.2, R31.2
- net MISO: now also P3.1 (P1)
- net MOSI: now also P3.4 (P4)
- net RES: now also P3.5 (P5)
- net SCK: now also P3.3 (P3)
- net VCC: now also P7.1 (P1)
- net at Q1.1 (G), R9.1: now also R28.2
- net at Q2.1 (G), R10.1: now also R29.1
- new net: R32.2, S1.1 (N)
- no-connect marks 16 -> 19
Other:
- moved on the sheet: Q1, Q2
